File: schematic/WirelessPalaSensor.sch (KiCad schematic (older format))
At the start: 18 parts, among them P1 USB_OTG, P2 SERIAL_TX, P3 Palazzetti Connector, SW1 RESET, SW2 RESCUE_MODE, U1 LM1117-3.3, U2 ESP-12, U3 DS18B20, U4 MCP4151-50k, U5 MCP4151-5k

Commit message: V3.2.3 Upgrade to Base V1.1.7
Parts:
- C1, C2: symbol CP -> Device:CP
- C3: symbol C -> Device:C
- D1: symbol LED_RGBW_SK6812 -> LED:SK6812
- P1: symbol USB_OTG -> Connector:USB_OTG
- P2, P3: symbol Conn_01x02 -> Connector_Generic:Conn_01x02
- R1, R2, R3, R4: symbol R -> Device:R
- SW1, SW2: symbol SW_Push -> Switch:SW_Push
- U1: symbol LM1117-3.3 -> Regulator_Linear:LM1117-3.3
- U2: symbol ESP-12 -> ESP8266:ESP-12
- U3: symbol DS18B20 -> maxim:DS18B20
- U4, U5: symbol MCP4151 -> DigiPot:MCP4151
Connections:
- wire segments 89 -> 98
Other:
- moved on the sheet: R4

Commit message: Update Schematic to D1 Mini
Parts:
- removed C1: 100uF, Capacitors_Tantalum_SMD:Tantalum_Case-B_EIA-3528-21_Hand, symbol Device:CP
- removed C2: 10uF, Capacitors_Tantalum_SMD:Tantalum_Case-A_EIA-3216-18_Hand, symbol Device:CP
- removed D1: SK6812, sk6812:Led_WS2812b, symbol LED:SK6812
- removed P1: USB_OTG, MicroUSB:MicroUSB, symbol Connector:USB_OTG
- removed P2: SERIAL_TX, Pin_Headers:Pin_Header_Straight_1x02_Pitch2.54mm, symbol Connector_Generic:Conn_01x02
- removed R3, R4: 10K, Resistors_SMD:R_0805_HandSoldering, symbol Device:R
- removed SW1: RESET, Buttons_Switches_ThroughHole:SW_PUSH_6mm, symbol Switch:SW_Push
- removed SW2: RESCUE_MODE, Buttons_Switches_ThroughHole:SW_PUSH_6mm, symbol Switch:SW_Push
- removed U1: LM1117-3.3, TO_SOT_Packages_SMD:SOT-223, symbol Regulator_Linear:LM1117-3.3
- removed U2: ESP-12, ESP8266:ESP12WithAdapter, symbol ESP8266:ESP-12
- added U1: WeMos_mini, wemos_d1_mini:wemos-d1-mini-DIL-only, symbol wemos_mini:WeMos_mini
Connections:
- wire segments 98 -> 65
Other:
- note removed: "ESP12F with \n2.54 adapter!"
- moved on the sheet: C3, P3, R1, R2, U3, U4, U5
