File: schematic/WirelessPalaSensor.kicad_pcb (KiCad board)
At the start: 2 copper layers, 25.4 x 29.8 mm, 8 parts, among them P3 Palazzetti Connector, U1 WeMos_mini, U3 DS18B20, U4 MCP4151-50k, U5 MCP4151-5k

Commit message: Update schematic to KiCAD8
Other:
- net class Default removed
